Commit message: Add Laser scan sensor to robot

File: src/m2wr_description/urdf/gazebo.xacro (robot description, xacro)
@@ -26,3 +26,34 @@
         </plugin>
     </gazebo>
+    <gazebo reference="sensor_laser">
+        <sensor type="ray" name="head_hokuyo_sensor">
+            <pose>0 0 0 0 0 0</pose>
+            <visualize>false</visualize>
+            <update_rate>40</update_rate>
+            <ray>
+                <scan>
+                    <horizontal>
+                        <samples>720</samples>
+                        <resolution>1</resolution>
+                        <min_angle>-3.141592</min_angle>
+                        <max_angle>3.141592</max_angle>
+                    </horizontal>
+                </scan>
+                <range>
+                    <min>0.10</min>
+                    <max>30.0</max>
+                    <resolution>0.01</resolution>
+                </range>
+                <noise>
+                    <type>gaussian</type>
+                    <mean>0.0</mean>
+                    <stddev>0.01</stddev>
+                </noise>
+            </ray>
+            <plugin name="gazebo_ros_head_hokuyo_controller" filename="libgazebo_ros_laser.so">
+                <topicName>/m2wr/laser/scan</topicName>
+                <frameName>sensor_laser</frameName>
+            </plugin>
+        </sensor>
+    </gazebo>
 </robot>

File: src/m2wr_description/urdf/m2wr.xacro (robot description, xacro)
@@ -55,3 +55,28 @@
     <xacro:link_wheel name="link_left_wheel" />
     <xacro:joint_wheel name="joint_left_wheel" child="link_left_wheel" origin_xyz="-0.05 -0.15 0" />
+    <link name="sensor_laser">
+        <inertial>
+            <origin xyz="0 0 0" rpy="0 0 0" />
+            <mass value="1" />
+            <xacro:cylinder_inertia mass="1" r="0.05" l="0.1" />
+        </inertial>
+        <visual>
+            <origin xyz="0 0 0" rpy="0 0 0" />
+            <geometry>
+                <cylinder radius="0.05" length="0.1"/>
+            </geometry>
+            <material name="white" />
+        </visual>
+        <collision>
+            <origin xyz="0 0 0" rpy="0 0 0"/>
+            <geometry>
+                <cylinder radius="0.05" length="0.1"/>
+            </geometry>
+        </collision>
+    </link>
+    <joint name="joint_sensor_laser" type="fixed">
+        <origin xyz="0.15 0 0.05" rpy="0 0 0"/>
+        <parent link="link_chassis"/>
+        <child link="sensor_laser"/>
+    </joint>
 </robot>

File: src/m2wr_description/urdf/macro.xacro (robot description, xacro)
@@ -1,4 +1,11 @@
 <?xml version="1.0"?>
+<!--
+  we will use macros, which are like functions, to reduce the remaining code in m2wr.xacro file.
+-->
 <robot xmlns:xacro="http://www.ros.org/wiki/xacro">
+    <!--
+      we have defined two macros, their purpose is to take parameters and create the required element (link element).
+      The first macro is named link_wheel and it accepts only one parameter name. It creates a wheel link with the name passed in the parameter.
+    -->
     <xacro:macro name="link_wheel" params="name">
         <link name="${name}">
@@ -22,4 +29,7 @@
         </link>
     </xacro:macro>
+    <!--
+      The second macro accepts three parameters name, child and origin_xyz and it creates a joint link.
+    -->
     <xacro:macro name="joint_wheel" params="name child origin_xyz">
         <joint name="${name}" type="continuous">
@@ -32,3 +42,9 @@
         </joint>
     </xacro:macro>
+    <!--
+      new macro for controlling the moment of inertia of the sensor cilinder
+    -->
+    <xacro:macro name="cylinder_inertia" params="mass r l">
+        <inertia ixx="${mass*(3*r*r+l*l)/12}" ixy = "0" ixz = "0" iyy="${mass*(3*r*r+l*l)/12}" iyz = "0" izz="${mass*(r*r)/2}" />
+    </xacro:macro>
 </robot>

Commit message: Update robot size

File: src/m2wr_description/urdf/gazebo.xacro (robot description, xacro)
@@ -18,5 +18,5 @@
             <rightJoint>joint_right_wheel</rightJoint>
             <wheelSeparation>0.4</wheelSeparation>
-            <wheelDiameter>0.2</wheelDiameter>
+            <wheelDiameter>0.14</wheelDiameter>
             <torque>0.1</torque>
             <commandTopic>cmd_vel</commandTopic>

File: src/m2wr_description/urdf/m2wr.xacro (robot description, xacro)
@@ -15,5 +15,5 @@
         <collision name="collision_chassis">
             <geometry>
-                <box size="0.5 0.3 0.07"/>
+                <box size="0.35 0.3 0.07"/>
             </geometry>
         </collision>
@@ -21,5 +21,5 @@
             <origin rpy="0 0 0" xyz="0 0 0"/>
             <geometry>
-                <box size="0.5 0.3 0.07"/>
+                <box size="0.35 0.3 0.07"/>
             </geometry>
             <material name="blue"/>
@@ -27,7 +27,7 @@
         <!-- caster front -->
         <collision name="caster_front_collision">
-            <origin rpy=" 0 0 0" xyz="0.35 0 -0.05"/>
+            <origin rpy=" 0 0 0" xyz="0.1 0 -0.035"/>
             <geometry>
-                <sphere radius="0.05"/>
+                <sphere radius="0.035"/>
             </geometry>
             <surface>
@@ -43,7 +43,7 @@
         </collision>
         <visual name="caster_front_visual">
-            <origin rpy=" 0 0 0" xyz="0.2 0 -0.05"/>
+            <origin rpy=" 0 0 0" xyz="0.1 0 -0.035"/>
             <geometry>
-                <sphere radius="0.05"/>
+                <sphere radius="0.035"/>
             </geometry>
         </visual>
@@ -76,5 +76,5 @@
     </link>
     <joint name="joint_sensor_laser" type="fixed">
-        <origin xyz="0.15 0 0.05" rpy="0 0 0"/>
+        <origin xyz="0.1 0 0.05" rpy="0 0 0"/>
         <parent link="link_chassis"/>
         <child link="sensor_laser"/>

File: src/m2wr_description/urdf/macro.xacro (robot description, xacro)
@@ -18,5 +18,5 @@
                 <origin rpy="0 1.5707 1.5707" xyz="0 0 0"/>
                 <geometry>
-                    <cylinder length="0.04" radius="0.1"/>
+                    <cylinder length="0.04" radius="0.07"/>
                 </geometry>
             </collision>
@@ -24,5 +24,5 @@
                 <origin rpy="0 1.5707 1.5707" xyz="0 0 0"/>
                 <geometry>
-                    <cylinder length="0.04" radius="0.1"/>
+                    <cylinder length="0.04" radius="0.07"/>
                 </geometry>
             </visual>

Commit message: Fixed robot model movement

File: src/m2wr_description/urdf/gazebo.xacro (robot description, xacro)
@@ -14,9 +14,9 @@
         <plugin filename="libgazebo_ros_diff_drive.so" name="differential_drive_controller">
             <alwaysOn>true</alwaysOn>
-            <updateRate>20</updateRate>
+            <updateRate>10</updateRate>
             <leftJoint>joint_left_wheel</leftJoint>
             <rightJoint>joint_right_wheel</rightJoint>
             <wheelSeparation>0.4</wheelSeparation>
-            <wheelDiameter>0.14</wheelDiameter>
+            <wheelDiameter>0.2</wheelDiameter>
             <torque>0.1</torque>
             <commandTopic>cmd_vel</commandTopic>

File: src/m2wr_description/urdf/m2wr.xacro (robot description, xacro)
@@ -15,5 +15,5 @@
         <collision name="collision_chassis">
             <geometry>
-                <box size="0.35 0.3 0.07"/>
+                <box size="0.5 0.3 0.07"/>
             </geometry>
         </collision>
@@ -21,5 +21,5 @@
             <origin rpy="0 0 0" xyz="0 0 0"/>
             <geometry>
-                <box size="0.35 0.3 0.07"/>
+                <box size="0.5 0.3 0.07"/>
             </geometry>
             <material name="blue"/>
@@ -27,7 +27,7 @@
         <!-- caster front -->
         <collision name="caster_front_collision">
-            <origin rpy=" 0 0 0" xyz="0.1 0 -0.035"/>
+            <origin rpy=" 0 0 0" xyz="0.35 0 -0.05"/>
             <geometry>
-                <sphere radius="0.035"/>
+                <sphere radius="0.05"/>
             </geometry>
             <surface>
@@ -43,7 +43,7 @@
         </collision>
         <visual name="caster_front_visual">
-            <origin rpy=" 0 0 0" xyz="0.1 0 -0.035"/>
+            <origin rpy=" 0 0 0" xyz="0.2 0 -0.05"/>
             <geometry>
-                <sphere radius="0.035"/>
+                <sphere radius="0.05"/>
             </geometry>
         </visual>
@@ -64,5 +64,5 @@
             <origin xyz="0 0 0" rpy="0 0 0" />
             <geometry>
-                <cylinder radius="0.05" length="0.1"/>
+                <cylinder radius="0.05" length="0.2"/>
             </geometry>
             <material name="white" />
@@ -76,5 +76,5 @@
     </link>
     <joint name="joint_sensor_laser" type="fixed">
-        <origin xyz="0.1 0 0.05" rpy="0 0 0"/>
+        <origin xyz="0.15 0 0.13" rpy="0 0 0"/>
         <parent link="link_chassis"/>
         <child link="sensor_laser"/>

File: src/m2wr_description/urdf/macro.xacro (robot description, xacro)
@@ -18,5 +18,5 @@
                 <origin rpy="0 1.5707 1.5707" xyz="0 0 0"/>
                 <geometry>
-                    <cylinder length="0.04" radius="0.07"/>
+                    <cylinder length="0.04" radius="0.1"/>
                 </geometry>
             </collision>
@@ -24,5 +24,5 @@
                 <origin rpy="0 1.5707 1.5707" xyz="0 0 0"/>
                 <geometry>
-                    <cylinder length="0.04" radius="0.07"/>
+                    <cylinder length="0.04" radius="0.1"/>
                 </geometry>
             </visual>
